File: ECAD/KinectIP.brd (EAGLE design)
At the start: 64.8 x 55.9 mm, 1 part

Commit message: update ECAD
Parts:
- added ID, PWR: RIGHT-ANGLE-SWITCH, Right-Angle-Switch:RIGHT-ANGLE-SWITCH
- added P5+: 2PIN-FEMALE-HEADER, Female-Header:2PIN-FEMALE-HEADER
Changed lines of the file:
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@@
 <setting verticaltext="up"/>
 </settings>
-<grid distance="50" unitdist="mil" unit="mil" style="lines" multiple="1" display="yes" altdistance="5" altunitdist="mil" altunit="mil"/>
+<grid distance="50" unitdist="mil" unit="mil" style="lines" multiple="1" display="yes" altdistance="1" altunitdist="mil" altunit="mil"/>
 <layers>
 <layer number="1" name="Top" color="4" fill="1" visible="yes" active="yes"/>
@@
 </layers>
 <board>
-<fusionsync huburn="a.cGVyc29uYWw6dWUyOGRkYTQ5" projecturn="a.cGVyc29uYWw6dWUyOGRkYTQ5IzIwMTkwNzIxMjA0NzU1MDc2" f3durn="urn:adsk.wipprod:dm.lineage:51sdf3HBRlSp9b0qTDdM7A" pcbguid="17f93904-f036-442f-8767-7531df551236" lastpulledtime="" lastsyncedchangeguid="6946e682-92d7-a103-ac63-fb9f0bad822b"/>
+<fusionsync huburn="a.cGVyc29uYWw6dWUyOGRkYTQ5" projecturn="a.cGVyc29uYWw6dWUyOGRkYTQ5IzIwMTkwNzIxMjA0NzU1MDc2" f3durn="urn:adsk.wipprod:dm.lineage:51sdf3HBRlSp9b0qTDdM7A" pcbguid="17f93904-f036-442f-8767-7531df551236" lastpulledtime="2019-07-25T10:40:12Z" lastsyncedchangeguid="28b22e7e-8deb-5dc0-aa3d-2cde74854504"/>
 <plain>
-<wire x1="0" y1="2.54" x2="0" y2="53.34" width="0.1524" layer="20"/>
-<wire x1="0" y1="53.34" x2="2.54" y2="55.88" width="0.1524" layer="20" curve="-90"/>
-<wire x1="2.54" y1="55.88" x2="62.23" y2="55.88" width="0.1524" layer="20"/>
-<wire x1="62.23" y1="55.88" x2="64.77" y2="53.34" width="0.1524" layer="20" curve="-90"/>
-<wire x1="64.77" y1="53.34" x2="64.77" y2="2.54" width="0.1524" layer="20"/>
-<wire x1="64.77" y1="2.54" x2="62.23" y2="0" width="0.1524" layer="20" curve="-90"/>
-<wire x1="62.23" y1="0" x2="2.54" y2="0" width="0.1524" layer="20"/>
-<wire x1="2.54" y1="0" x2="0" y2="2.54" width="0.1524" layer="20" curve="-90"/>
+<wire x1="2.54" y1="55.88" x2="0" y2="53.34" width="0.254" layer="20" curve="90"/>
+<wire x1="0" y1="53.34" x2="0" y2="2.54" width="0.254" layer="20"/>
+<wire x1="0" y1="2.54" x2="2.54" y2="0" width="0.254" layer="20" curve="90"/>
+<wire x1="2.54" y1="0" x2="62.23" y2="0" width="0.254" layer="20"/>
+<wire x1="62.23" y1="0" x2="64.77" y2="2.54" width="0.254" layer="20" curve="90"/>
+<wire x1="64.77" y1="2.54" x2="64.77" y2="53.34" width="0.254" layer="20"/>
+<wire x1="64.77" y1="53.34" x2="62.23" y2="55.88" width="0.254" layer="20" curve="90"/>
+<wire x1="62.23" y1="55.88" x2="2.54" y2="55.88" width="0.254" layer="20"/>
 </plain>
 <attributes>
@@
 </autorouter>
 <elements>
-<element name="PCB2" library="Rock64" package="ROCK64" package3d_urn="urn:adsk.eagle:package:12239992/2" value="ROCK64ROCK64" x="0" y="0" smashed="yes"/>
+<element name="PCB2" library="Rock64" package="ROCK64" package3d_urn="urn:adsk.eagle:package:12239992/2" value="ROCK64ROCK64" x="0" y="0" locked="yes" smashed="yes"/>
+<element name="PWR" library="Right-Angle-Switch" package="RIGHT-ANGLE-SWITCH" package3d_urn="urn:adsk.eagle:package:12341458/3" value="RIGHT-ANGLE-SWITCH" x="44.45" y="2.54" smashed="yes" rot="MR180">
+<attribute name="NAME" x="39.45" y="7.54" size="1.27" layer="26" rot="MR270"/>
+<attribute name="VALUE" x="50.7" y="7.54" size="1.27" layer="26" rot="MR270"/>
+</element>
+<element name="ID" library="Right-Angle-Switch" package="RIGHT-ANGLE-SWITCH" package3d_urn="urn:adsk.eagle:package:12341458/3" value="RIGHT-ANGLE-SWITCH" x="20.32" y="2.54" smashed="yes" rot="MR180">
+<attribute name="NAME" x="15.32" y="7.54" size="1.27" layer="26" rot="MR270"/>
+<attribute name="VALUE" x="26.57" y="7.54" size="1.27" layer="26" rot="MR270"/>
+</element>
+<element name="P5+" library="Female-Header" package="2PIN-FEMALE-HEADER" package3d_urn="urn:adsk.eagle:package:12344424/3" value="2PIN-FEMALE-HEADER" x="16.255" y="48.155" locked="yes" smashed="yes" rot="MR180">
+<attribute name="NAME" x="20.954" y="48.917" size="1.016" layer="22" rot="MR180"/>
+</element>
 </elements>
 <signals>

Commit message: add lbr
Parts:
- added LED1: (no value), led:LED3MM
- added R1, R4, R5: 330R, rcl:R0805
- added R2, R3: 10K, rcl:R0805
- moved PCB2 5.08 mm to (0.00, 5.08)
- moved P5+ 5.08 mm to (16.3, 53.2)
- moved ID 2.13 mm to (18.4, 3.49)
- moved PWR 1.14 mm to (43.8, 3.49)
Connections:
- new net +3V3: PCB2.P$1, R4.2, R5.2
- new net 0V: ID.MNT$1, ID.MNT$2, PCB2.P$25, PWR.MNT$1, PWR.MNT$2, R1.1, R2.1, R3.1
- new net N$1: LED1.A, PCB2.P$15
- new net N$2: LED1.K, R1.2
- new net N$3: ID.SW$2, R4.1
- new net N$4: PWR.SW$2, R5.1
- new net N$5: ID.SW$1, P5+.P$1, R2.2
- new net N$6: P5+.P$2, PWR.SW$1, R3.2
Other:
- board size 64.8 x 55.9 mm -> 64.8 x 60 mm

Commit message: managed lib
Parts:
- added J1: (no value), con-jack-3D:SPC4077
Connections:
- new net +12V: J1.3
- net 0V: now also J1.1, J1.2
Changed lines of the file:
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@@
 <drawing>
 <settings>
-<setting alwaysvectorfont="yes"/>
+<setting alwaysvectorfont="no"/>
 <setting verticaltext="up"/>
 </settings>
@@
 <layer number="44" name="Drills" color="7" fill="1" visible="no" active="yes"/>
 <layer number="45" name="Holes" color="7" fill="1" visible="no" active="yes"/>
-<layer number="46" name="Milling" color="3" fill="1" visible="no" active="yes"/>
+<layer number="46" name="Milling" color="3" fill="1" visible="yes" active="yes"/>
 <layer number="47" name="Measures" color="7" fill="1" visible="no" active="yes"/>
 <layer number="48" name="Document" color="7" fill="1" visible="yes" active="yes"/>
@@
 </autorouter>
 <elements>
-<element name="PCB2" library="Rock64" package="ROCK64" package3d_urn="urn:adsk.eagle:package:12239992/2" value="ROCK64ROCK64" x="0" y="5.08" smashed="yes"/>
-<element name="PWR" library="Right-Angle-Switch" package="RIGHT-ANGLE-SWITCH" package3d_urn="urn:adsk.eagle:package:12341458/3" value="RIGHT-ANGLE-SWITCH" x="43.815" y="3.4925" smashed="yes" rot="MR180">
+<element name="PCB2" library="Rock64" library_urn="urn:adsk.eagle:library:12241252" package="ROCK64" package3d_urn="urn:adsk.eagle:package:12239992/2" value="ROCK64ROCK64" x="0" y="5.08" smashed="yes"/>
+<element name="PWR" library="Right-Angle-Switch" library_urn="urn:adsk.eagle:library:12341455" package="RIGHT-ANGLE-SWITCH" package3d_urn="urn:adsk.eagle:package:12341458/3" value="RIGHT-ANGLE-SWITCH" x="43.815" y="3.4925" smashed="yes" rot="MR180">
 <attribute name="NAME" x="38.815" y="8.4925" size="1.27" layer="26" rot="MR270"/>
 <attribute name="VALUE" x="50.065" y="8.4925" size="1.27" layer="26" rot="MR270"/>
 </element>
-<element name="ID" library="Right-Angle-Switch" package="RIGHT-ANGLE-SWITCH" package3d_urn="urn:adsk.eagle:package:12341458/3" value="RIGHT-ANGLE-SWITCH" x="18.415" y="3.4925" smashed="yes" rot="MR180">
+<element name="ID" library="Right-Angle-Switch" library_urn="urn:adsk.eagle:library:12341455" package="RIGHT-ANGLE-SWITCH" package3d_urn="urn:adsk.eagle:package:12341458/3" value="RIGHT-ANGLE-SWITCH" x="18.415" y="3.4925" smashed="yes" rot="MR180">
 <attribute name="NAME" x="13.415" y="8.4925" size="1.27" layer="26" rot="MR270"/>
 <attribute name="VALUE" x="24.665" y="8.4925" size="1.27" layer="26" rot="MR270"/>
 </element>
-<element name="P5+" library="Female-Header" package="2PIN-FEMALE-HEADER" package3d_urn="urn:adsk.eagle:package:12344424/3" value="2PIN-FEMALE-HEADER" x="16.255" y="53.235" smashed="yes" rot="MR180">
+<element name="P5+" library="Female-Header" library_urn="urn:adsk.eagle:library:12344421" package="2PIN-FEMALE-HEADER" package3d_urn="urn:adsk.eagle:package:12344424/3" value="2PIN-FEMALE-HEADER" x="16.255" y="53.235" smashed="yes" rot="MR180">
 <attribute name="NAME" x="20.954" y="53.997" size="1.016" layer="22" rot="MR180"/>
 </element>
 <element name="LED1" library="led" library_urn="urn:adsk.eagle:library:259" package="LED3MM" package3d_urn="urn:adsk.eagle:package:15797/1" value="" x="31.4325" y="3.4925" smashed="yes">
 <attribute name="NAME" x="33.3375" y="3.8735" size="1.27" layer="25" ratio="10"/>
+<attribute name="POPULARITY" value="97" x="31.4325" y="3.4925" size="1.778" layer="27" display="off"/>
 <attribute name="VALUE" x="33.3375" y="1.8415" size="1.27" layer="27" ratio="10"/>
 </element>
 <element name="R1" library="rcl" library_urn="urn:adsk.eagle:library:334" package="R0805" package3d_urn="urn:adsk.eagle:package:23553/2" value="330R" x="35.56" y="4.445" smashed="yes" rot="R270">
 <attribute name="NAME" x="36.83" y="5.08" size="1.27" layer="25" rot="R270"/>
+<attribute name="POPULARITY" value="86" x="35.56" y="4.445" size="1.778" layer="27" rot="R270" display="off"/>
 <attribute name="SPICEPREFIX" value="R" x="35.56" y="4.445" size="1.778" layer="27" rot="R270" display="off"/>
 <attribute name="VALUE" x="33.02" y="5.08" size="1.27" layer="27" rot="R270"/>
@@
 <element name="R2" library="rcl" library_urn="urn:adsk.eagle:library:334" package="R0805" package3d_urn="urn:adsk.eagle:package:23553/2" value="10K" x="17.145" y="10.4775" smashed="yes" rot="R270">
 <attribute name="NAME" x="18.415" y="11.1125" size="1.27" layer="25" rot="R270"/>
+<attribute name="POPULARITY" value="86" x="17.145" y="10.4775" size="1.778" layer="27" rot="R270" display="off"/>
 <attribute name="SPICEPREFIX" value="R" x="17.145" y="10.4775" size="1.778" layer="27" rot="R270" display="off"/>
 <attribute name="VALUE" x="14.605" y="11.1125" size="1.27" layer="27" rot="R270"/>
@@
 <element name="R3" library="rcl" library_urn="urn:adsk.eagle:library:334" package="R0805" package3d_urn="urn:adsk.eagle:package:23553/2" value="10K" x="42.545" y="10.4775" smashed="yes" rot="R270">
 <attribute name="NAME" x="43.815" y="11.1125" size="1.27" layer="25" rot="R270"/>
+<attribute name="POPULARITY" value="86" x="42.545" y="10.4775" size="1.778" layer="27" rot="R270" display="off"/>
 <attribute name="SPICEPREFIX" value="R" x="42.545" y="10.4775" size="1.778" layer="27" rot="R270" display="off"/>
 <attribute name="VALUE" x="40.005" y="11.1125" size="1.27" layer="27" rot="R270"/>
@@
 <element name="R4" library="rcl" library_urn="urn:adsk.eagle:library:334" package="R0805" package3d_urn="urn:adsk.eagle:package:23553/2" value="330R" x="19.685" y="10.4775" smashed="yes" rot="R90">
 <attribute name="NAME" x="18.415" y="9.8425" size="1.27" layer="25" rot="R90"/>
+<attribute name="POPULARITY" value="86" x="19.685" y="10.4775" size="1.778" layer="27" rot="R90" display="off"/>
 <attribute name="SPICEPREFIX" value="R" x="19.685" y="10.4775" size="1.778" layer="27" rot="R90" display="off"/>
 <attribute name="VALUE" x="22.225" y="9.8425" size="1.27" layer="27" rot="R90"/>
@@
 <element name="R5" library="rcl" library_urn="urn:adsk.eagle:library:334" package="R0805" package3d_urn="urn:adsk.eagle:package:23553/2" value="330R" x="45.085" y="10.4775" smashed="yes" rot="R90">
 <attribute name="NAME" x="43.815" y="9.8425" size="1.27" layer="25" rot="R90"/>
+<attribute name="POPULARITY" value="86" x="45.085" y="10.4775" size="1.778" layer="27" rot="R90" display="off"/>
 <attribute name="SPICEPREFIX" value="R" x="45.085" y="10.4775" size="1.778" layer="27" rot="R90" display="off"/>
 <attribute name="VALUE" x="47.625" y="9.8425" size="1.27" layer="27" rot="R90"/>
+</element>
+<element name="J1" library="con-jack-3D" library_urn="urn:adsk.eagle:library:12345140" package="SPC4077" package3d_urn="urn:adsk.eagle:package:12345148/2" value="" x="11.1125" y="18.415" smashed="yes" rot="MR180">
+<attribute name="MF" value="" x="11.1125" y="18.415" size="1.778" layer="28" rot="MR180" display="off"/>
+<attribute name="MPN" value="" x="11.1125" y="18.415" size="1.778" layer="28" rot="MR180" display="off"/>
+<attribute name="NAME" x="0.9525" y="13.335" size="1.27" layer="26" rot="MR180"/>
+<attribute name="OC_FARNELL" value="unknown" x="11.1125" y="18.415" size="1.778" layer="28" rot="MR180" display="off"/>
+<attribute name="OC_NEWARK" value="unknown" x="11.1125" y="18.415" size="1.778" layer="28" rot="MR180" display="off"/>
+<attribute name="VALUE" x="0.9525" y="24.765" size="1.27" layer="28" rot="MR180"/>
 </element>
 </elements>
@@
 <contactref element="PWR" pad="MNT$2"/>
 <contactref element="PCB2" pad="P$25"/>
+<contactref element="J1" pad="1"/>
+<contactref element="J1" pad="2"/>
 <wire x1="42.545" y1="11.4275" x2="38.8366" y2="56.3118" width="0" layer="19" extent="1-1"/>
 <wire x1="40.065" y1="6.2425" x2="42.545" y2="11.4275" width="0" layer="19" extent="1-1"/>
@@
 <wire x1="17.145" y1="11.4275" x2="22.165" y2="6.2425" width="0" layer="19" extent="1-1"/>
 <wire x1="14.665" y1="6.2425" x2="17.145" y2="11.4275" width="0" layer="19" extent="1-1"/>
+<wire x1="8.1125" y1="18.415" x2="14.665" y2="6.2425" width="0" layer="19" extent="1-1"/>
+<wire x1="11.1125" y1="23.215" x2="8.1125" y2="18.415" width="0" layer="19" extent="1-1"/>
 </signal>
 <signal name="N$1">
@@
 <wire x1="41.565" y1="3.4925" x2="42.545" y2="9.5275" width="0" layer="19" extent="1-1"/>
 </signal>
+<signal name="+12V">
+<contactref element="J1" pad="3"/>
+</signal>
 </signals>

Commit message: LED Lib
Parts:
- removed LED1: (no value), led:LED3MM
- added C1: (no value), rcl:C0805K
- added LED: BLUE, LED-90-Degree:LED-90-DEG
- moved J1 15.1 mm to (5.40, 32.4)
- moved R1 8.72 mm to (27.0, 6.03)
Connections:
- net N$1: now also LED.A; no longer LED1.A
- net N$2: now also LED.K; no longer LED1.K
Changed lines of the file:
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@@
 <drawing>
 <settings>
-<setting alwaysvectorfont="no"/>
+<setting alwaysvectorfont="yes"/>
 <setting verticaltext="up"/>
 </settings>
@@
 </layers>
 <board>
-<fusionsync huburn="a.cGVyc29uYWw6dWUyOGRkYTQ5" projecturn="a.cGVyc29uYWw6dWUyOGRkYTQ5IzIwMTkwNzIxMjA0NzU1MDc2" f3durn="urn:adsk.wipprod:dm.lineage:51sdf3HBRlSp9b0qTDdM7A" pcbguid="17f93904-f036-442f-8767-7531df551236" lastpulledtime="2019-07-25T10:40:12Z" lastsyncedchangeguid="a1cbfe57-5863-5e82-e509-078602fa2d75"/>
+<fusionsync huburn="a.cGVyc29uYWw6dWUyOGRkYTQ5" projecturn="a.cGVyc29uYWw6dWUyOGRkYTQ5IzIwMTkwNzIxMjA0NzU1MDc2" f3durn="urn:adsk.wipprod:dm.lineage:51sdf3HBRlSp9b0qTDdM7A" pcbguid="17f93904-f036-442f-8767-7531df551236" lastpulledtime="2019-07-25T10:40:12Z" lastsyncedchangeguid="30b88b88-6244-209e-32c0-b88ed1906c49"/>
 <plain>
 <wire x1="2.54" y1="60.96" x2="0" y2="58.42" width="0.254" layer="20" curve="90"/>
@@
 <attribute name="NAME" x="20.954" y="53.997" size="1.016" layer="22" rot="MR180"/>
 </element>
-<element name="LED1" library="led" library_urn="urn:adsk.eagle:library:259" package="LED3MM" package3d_urn="urn:adsk.eagle:package:15797/1" value="" x="31.4325" y="3.4925" smashed="yes">
-<attribute name="NAME" x="33.3375" y="3.8735" size="1.27" layer="25" ratio="10"/>
-<attribute name="POPULARITY" value="97" x="31.4325" y="3.4925" size="1.778" layer="27" display="off"/>
-<attribute name="VALUE" x="33.3375" y="1.8415" size="1.27" layer="27" ratio="10"/>
-</element>
-<element name="R1" library="rcl" library_urn="urn:adsk.eagle:library:334" package="R0805" package3d_urn="urn:adsk.eagle:package:23553/2" value="330R" x="35.56" y="4.445" smashed="yes" rot="R270">
-<attribute name="NAME" x="36.83" y="5.08" size="1.27" layer="25" rot="R270"/>
-<attribute name="POPULARITY" value="86" x="35.56" y="4.445" size="1.778" layer="27" rot="R270" display="off"/>
-<attribute name="SPICEPREFIX" value="R" x="35.56" y="4.445" size="1.778" layer="27" rot="R270" display="off"/>
-<attribute name="VALUE" x="33.02" y="5.08" size="1.27" layer="27" rot="R270"/>
+<element name="R1" library="rcl" library_urn="urn:adsk.eagle:library:334" package="R0805" package3d_urn="urn:adsk.eagle:package:23553/2" value="330R" x="26.9875" y="6.0325" smashed="yes" rot="R270">
+<attribute name="NAME" x="28.2575" y="6.6675" size="1.27" layer="25" rot="R270"/>
+<attribute name="POPULARITY" value="86" x="26.9875" y="6.0325" size="1.778" layer="27" rot="R270" display="off"/>
+<attribute name="SPICEPREFIX" value="R" x="26.9875" y="6.0325" size="1.778" layer="27" rot="R270" display="off"/>
+<attribute name="VALUE" x="24.4475" y="6.6675" size="1.27" layer="27" rot="R270"/>
 </element>
 <element name="R2" library="rcl" library_urn="urn:adsk.eagle:library:334" package="R0805" package3d_urn="urn:adsk.eagle:package:23553/2" value="10K" x="17.145" y="10.4775" smashed="yes" rot="R270">
@@
 <attribute name="VALUE" x="47.625" y="9.8425" size="1.27" layer="27" rot="R90"/>
 </element>
-<element name="J1" library="con-jack-3D" library_urn="urn:adsk.eagle:library:12345140" package="SPC4077" package3d_urn="urn:adsk.eagle:package:12345148/2" value="" x="11.1125" y="18.415" smashed="yes" rot="MR180">
-<attribute name="MF" value="" x="11.1125" y="18.415" size="1.778" layer="28" rot="MR180" display="off"/>
-<attribute name="MPN" value="" x="11.1125" y="18.415" size="1.778" layer="28" rot="MR180" display="off"/>
-<attribute name="NAME" x="0.9525" y="13.335" size="1.27" layer="26" rot="MR180"/>
-<attribute name="OC_FARNELL" value="unknown" x="11.1125" y="18.415" size="1.778" layer="28" rot="MR180" display="off"/>
-<attribute name="OC_NEWARK" value="unknown" x="11.1125" y="18.415" size="1.778" layer="28" rot="MR180" display="off"/>
-<attribute name="VALUE" x="0.9525" y="24.765" size="1.27" layer="28" rot="MR180"/>
+<element name="J1" library="con-jack-3D" library_urn="urn:adsk.eagle:library:12345140" package="SPC4077" package3d_urn="urn:adsk.eagle:package:12345148/2" value="" x="5.3975" y="32.385" smashed="yes" rot="MR180">
+<attribute name="MF" value="" x="5.3975" y="32.385" size="1.778" layer="28" rot="MR180" display="off"/>
+<attribute name="MPN" value="" x="5.3975" y="32.385" size="1.778" layer="28" rot="MR180" display="off"/>
+<attribute name="NAME" x="-4.7625" y="27.305" size="1.27" layer="26" rot="MR180"/>
+<attribute name="OC_FARNELL" value="unknown" x="5.3975" y="32.385" size="1.778" layer="28" rot="MR180" display="off"/>
+<attribute name="OC_NEWARK" value="unknown" x="5.3975" y="32.385" size="1.778" layer="28" rot="MR180" display="off"/>
+<attribute name="VALUE" x="-4.7625" y="38.735" size="1.27" layer="28" rot="MR180"/>
+</element>
+<element name="LED" library="LED-90-Degree" library_urn="urn:adsk.eagle:library:12346089" package="LED-90-DEG" package3d_urn="urn:adsk.eagle:package:12346092/4" value="BLUE" x="31.115" y="5.08" smashed="yes" rot="MR0">
+<attribute name="NAME" x="33.7185" y="2.2225" size="1.27" layer="26" ratio="10" rot="MR90"/>
+<attribute name="VALUE" x="27.559" y="1.905" size="1.27" layer="28" ratio="10" rot="MR90"/>
+</element>
+<element name="C1" library="rcl" library_urn="urn:adsk.eagle:library:334" package="C0805K" package3d_urn="urn:adsk.eagle:package:23681/2" value="" x="-3.4925" y="-14.605" smashed="yes">
+<attribute name="NAME" x="-4.4925" y="-13.73" size="1.016" layer="25"/>
+<attribute name="POPULARITY" value="52" x="-3.4925" y="-14.605" size="1.778" layer="27" display="off"/>
+<attribute name="SPICEPREFIX" value="C" x="-3.4925" y="-14.605" size="1.778" layer="27" display="off"/>
+<attribute name="VALUE" x="-4.4925" y="-16.505" size="1.016" layer="27"/>
 </element>
 </elements>
@@
 <wire x1="42.545" y1="11.4275" x2="38.8366" y2="56.3118" width="0" layer="19" extent="1-1"/>
 <wire x1="40.065" y1="6.2425" x2="42.545" y2="11.4275" width="0" layer="19" extent="1-1"/>
-<wire x1="35.56" y1="5.395" x2="40.065" y2="6.2425" width="0" layer="19" extent="1-1"/>
+<wire x1="26.9875" y1="6.9825" x2="40.065" y2="6.2425" width="0" layer="19" extent="1-1"/>
 <wire x1="47.565" y1="6.2425" x2="42.545" y2="11.4275" width="0" layer="19" extent="1-1"/>
-<wire x1="22.165" y1="6.2425" x2="35.56" y2="5.395" width="0" layer="19" extent="1-1"/>
+<wire x1="22.165" y1="6.2425" x2="26.9875" y2="6.9825" width="0" layer="19" extent="1-1"/>
 <wire x1="17.145" y1="11.4275" x2="22.165" y2="6.2425" width="0" layer="19" extent="1-1"/>
 <wire x1="14.665" y1="6.2425" x2="17.145" y2="11.4275" width="0" layer="19" extent="1-1"/>
-<wire x1="8.1125" y1="18.415" x2="14.665" y2="6.2425" width="0" layer="19" extent="1-1"/>
-<wire x1="11.1125" y1="23.215" x2="8.1125" y2="18.415" width="0" layer="19" extent="1-1"/>
+<wire x1="2.3975" y1="32.385" x2="14.665" y2="6.2425" width="0" layer="19" extent="1-1"/>
+<wire x1="5.3975" y1="37.185" x2="2.3975" y2="32.385" width="0" layer="19" extent="1-1"/>
 </signal>
 <signal name="N$1">
 <contactref element="PCB2" pad="P$15"/>
-<contactref element="LED1" pad="A"/>
-<wire x1="30.1625" y1="3.4925" x2="26.1366" y2="56.3118" width="0" layer="19" extent="1-1"/>
+<contactref element="LED" pad="A"/>
+<wire x1="32.385" y1="5.08" x2="26.1366" y2="56.3118" width="0" layer="19" extent="1-1"/>
 </signal>
 <signal name="N$2">
-<contactref element="LED1" pad="K"/>
 <contactref element="R1" pad="2"/>
-<wire x1="32.7025" y1="3.4925" x2="35.56" y2="3.495" width="0" layer="19" extent="1-1"/>
+<contactref element="LED" pad="K"/>
+<wire x1="29.845" y1="5.08" x2="26.9875" y2="5.0825" width="0" layer="19" extent="1-1"/>
 </signal>
 <signal name="N$3">
