File: ECAD/KinectIP.brd (EAGLE design)
At the start: 64.8 x 59.4 mm, 13 parts, among them P5+ 2PIN-FEMALE-HEADER

Commit message: update ECAD
Parts:
- added KINECT_BLACK, KINECT_BROWN, KINECT_GREY, USB3_BLUE, USB3_GND1, USB3_GND2, USB3_ORANGE, USB3_PURPLE, USB3_YELLOW, USB_D+, USB_D-, USB_GND, USB_VCC: (no value), wirepad:SMD1,27-2,54
- added SH1, SH2: GND, wirepad:SMD2,54-5,08
- moved J1 74.3 mm to (75.9, 8.89), turned to 0 degrees
- moved 12V->5V 30.8 mm to (60.3, 45.1), turned to 270 degrees
- moved C1 10.4 mm to (5.71, 61.3), turned to 270 degrees
- moved P5+ 8.89 mm to (16.3, 62.1)
- moved PCB2 8.89 mm to (0.00, 14.0)
Connections:
- net +12V: now also KINECT_BROWN.1
- net 0V: now also KINECT_BLACK.1, KINECT_GREY.1, SH1.1, SH2.1
Other:
- board size 64.8 x 59.4 mm -> 81.3 x 68.3 mm

Commit message: ecad update
Parts:
- added PAD1, PAD2, PAD3, PAD4: (no value), wirepad:1,6/0,8
- added U$1: BOJIT_COPPER, BOJIT Logos:BOJIT_LARGE_COPPER
- added USB3_BLUE_HOST, USB3_GND1_HOST, USB3_GND2_HOST, USB3_ORANGE_HOST, USB3_PURPLE_HOST, USB3_YELLOW_HOST, USB_D+_HOST, USB_D-_HOST, USB_GND_HOST, USB_VCC_HOST: (no value), wirepad:SMD1,27-2,54
- moved 12V->5V 6.99 mm to (60.0, 52.1), turned to 90 degrees
- moved C1 5.54 mm to (10.8, 59.1)
- moved KINECT_BLACK 1.27 mm to (34.9, 41.9)
- moved KINECT_BROWN 1.27 mm to (34.9, 44.5)
- moved KINECT_GREY 1.27 mm to (34.9, 39.4)
Connections:
- new net N$10: USB_GND.1, USB_GND_HOST.1
- new net N$11: USB3_ORANGE.1, USB3_ORANGE_HOST.1
- new net N$12: USB3_PURPLE.1, USB3_PURPLE_HOST.1
- new net N$13: USB3_GND1.1, USB3_GND1_HOST.1, USB3_GND2.1, USB3_GND2_HOST.1
- new net N$15: USB3_YELLOW.1, USB3_YELLOW_HOST.1
- new net N$16: USB3_BLUE.1, USB3_BLUE_HOST.1
- new net N$7: USB_VCC.1, USB_VCC_HOST.1
- new net N$8: USB_D-.1, USB_D-_HOST.1
- new net N$9: USB_D+.1, USB_D+_HOST.1
Routing:
- net +3V3: track 0.00 -> 93.8 mm
- net N$6: track 0.00 -> 85.6 mm
- net +12V: track 0.00 -> 70.0 mm
- net N$5: track 0.00 -> 65.9 mm
- net N$1: track 0.00 -> 64.3 mm
- net +5V: track 0.00 -> 61.5 mm
- net N$13: track 0.00 -> 33.5 mm
- net N$11: track 0.00 -> 33.4 mm
- net N$12: track 0.00 -> 25.8 mm
- net N$10: track 0.00 -> 25.3 mm
- net N$9: track 0.00 -> 24.7 mm
- net N$7: track 0.00 -> 24.5 mm
- net N$8: track 0.00 -> 24.4 mm
- net N$15: track 0.00 -> 18.6 mm
- net N$16: track 0.00 -> 8.78 mm
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- added copper zone on layer 1, net +5V
- added copper zone on layer 1, net 0V
- added copper zone on layer 16, net 0V
- added copper zone on layer 16, net 0V1
Other:
- outline, holes or cut-outs redrawn
- board text added: "USB3"
