File: ECAD/KinectIP.sch (EAGLE design)
At the start: 4 parts, among them P5+ 2PIN-FEMALE-HEADER

Commit message: add lbr
Parts:
- added LED1: (no value), led:LED3MM
- added R1, R4, R5: 330R, rcl:R-EU_R0805
- added R2, R3: 10K, rcl:R-EU_R0805
Connections:
- new net +3V3: PCB2.3V3@1, R4.2, R5.2
- new net 0V: ID.MNT$1, ID.MNT$2, PCB2.GND@25, PWR.MNT$1, PWR.MNT$2, R1.1, R2.1, R3.1
- new net N$1: LED1.A, PCB2.GPIO22
- new net N$2: LED1.C, R1.2
- new net N$3: ID.SW$2, R4.1
- new net N$4: PWR.SW$2, R5.1
- new net N$5: ID.SW$1, P5+.P$1, R2.2
- new net N$6: P5+.P$2, PWR.SW$1, R3.2
Other:
- note added: "P5+ GPIO"
- moved on the sheet: ID, PWR

Commit message: managed lib
Parts:
- added J1: (no value), con-jack-3D:JACK-PLUG-SLOTTED0
Connections:
- new net +12V: J1.3
- net 0V: now also J1.1, J1.2
Changed lines of the file:
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@@
 </classes>
 <parts>
-<part name="PCB2" library="Rock64" deviceset="ROCK64" device="ROCK64" package3d_urn="urn:adsk.eagle:package:12239992/2"/>
-<part name="PWR" library="Right-Angle-Switch" deviceset="RIGHT-ANGLE-SWITCH" device="" package3d_urn="urn:adsk.eagle:package:12341458/3"/>
-<part name="ID" library="Right-Angle-Switch" deviceset="RIGHT-ANGLE-SWITCH" device="" package3d_urn="urn:adsk.eagle:package:12341458/3"/>
-<part name="P5+" library="Female-Header" deviceset="2PIN-FEMALE-HEADER" device="" package3d_urn="urn:adsk.eagle:package:12344424/3"/>
+<part name="PCB2" library="Rock64" library_urn="urn:adsk.eagle:library:12241252" deviceset="ROCK64" device="ROCK64" package3d_urn="urn:adsk.eagle:package:12239992/2"/>
+<part name="PWR" library="Right-Angle-Switch" library_urn="urn:adsk.eagle:library:12341455" deviceset="RIGHT-ANGLE-SWITCH" device="" package3d_urn="urn:adsk.eagle:package:12341458/3"/>
+<part name="ID" library="Right-Angle-Switch" library_urn="urn:adsk.eagle:library:12341455" deviceset="RIGHT-ANGLE-SWITCH" device="" package3d_urn="urn:adsk.eagle:package:12341458/3"/>
+<part name="P5+" library="Female-Header" library_urn="urn:adsk.eagle:library:12344421" deviceset="2PIN-FEMALE-HEADER" device="" package3d_urn="urn:adsk.eagle:package:12344424/3"/>
 <part name="LED1" library="led" library_urn="urn:adsk.eagle:library:259" deviceset="LED" device="3MM" package3d_urn="urn:adsk.eagle:package:15797/1"/>
 <part name="R1" library="rcl" library_urn="urn:adsk.eagle:library:334" deviceset="R-EU_" device="R0805" package3d_urn="urn:adsk.eagle:package:23553/2" value="330R"/>
@@
 <part name="R4" library="rcl" library_urn="urn:adsk.eagle:library:334" deviceset="R-EU_" device="R0805" package3d_urn="urn:adsk.eagle:package:23553/2" value="330R"/>
 <part name="R5" library="rcl" library_urn="urn:adsk.eagle:library:334" deviceset="R-EU_" device="R0805" package3d_urn="urn:adsk.eagle:package:23553/2" value="330R"/>
+<part name="J1" library="con-jack-3D" library_urn="urn:adsk.eagle:library:12345140" deviceset="JACK-PLUG-SLOTTED" device="0" package3d_urn="urn:adsk.eagle:package:12345148/2"/>
 </parts>
 <sheets>
@@
 <attribute name="VALUE" x="175.895" y="66.04" size="1.778" layer="96"/>
 </instance>
-<instance part="P+1" gate="1" x="114.3" y="187.96" smashed="yes">
-<attribute name="VALUE" x="111.76" y="182.88" size="1.778" layer="96" rot="R90"/>
-</instance>
-<instance part="P+2" gate="1" x="93.98" y="187.96" smashed="yes">
-<attribute name="VALUE" x="91.44" y="182.88" size="1.778" layer="96" rot="R90"/>
+<instance part="P+1" gate="1" x="116.84" y="162.56" smashed="yes">
+<attribute name="VALUE" x="114.3" y="157.48" size="1.778" layer="96" rot="R90"/>
+</instance>
+<instance part="P+2" gate="1" x="88.9" y="162.56" smashed="yes">
+<attribute name="VALUE" x="86.36" y="157.48" size="1.778" layer="96" rot="R90"/>
 </instance>
 <instance part="R4" gate="G$1" x="147.32" y="137.16" smashed="yes" rot="R90">
@@
 <attribute name="NAME" x="163.6014" y="133.35" size="1.778" layer="95" rot="R90"/>
 <attribute name="VALUE" x="168.402" y="133.35" size="1.778" layer="96" rot="R90"/>
+</instance>
+<instance part="J1" gate="G$1" x="78.74" y="152.4" smashed="yes">
+<attribute name="NAME" x="71.12" y="157.48" size="1.778" layer="95"/>
+<attribute name="VALUE" x="71.12" y="147.32" size="1.778" layer="96"/>
 </instance>
 </instances>
@@
 <pinref part="PCB2" gate="G$1" pin="GND@25"/>
 <wire x1="269.24" y1="129.54" x2="269.24" y2="152.4" width="0.1524" layer="91"/>
+<pinref part="J1" gate="G$1" pin="1"/>
+<wire x1="83.82" y1="149.86" x2="88.9" y2="149.86" width="0.1524" layer="91"/>
+<wire x1="88.9" y1="149.86" x2="88.9" y2="71.12" width="0.1524" layer="91"/>
+<wire x1="88.9" y1="71.12" x2="134.62" y2="71.12" width="0.1524" layer="91"/>
+<junction x="134.62" y="71.12"/>
+<pinref part="J1" gate="G$1" pin="2"/>
+<wire x1="83.82" y1="152.4" x2="88.9" y2="152.4" width="0.1524" layer="91"/>
+<wire x1="88.9" y1="152.4" x2="88.9" y2="149.86" width="0.1524" layer="91"/>
+<junction x="88.9" y="149.86"/>
 </segment>
 </net>
@@
 </segment>
 </net>
+<net name="+12V" class="0">
+<segment>
+<pinref part="J1" gate="G$1" pin="3"/>
+<pinref part="P+2" gate="1" pin="+12V"/>
+<wire x1="83.82" y1="154.94" x2="88.9" y2="154.94" width="0.1524" layer="91"/>
+<wire x1="88.9" y1="154.94" x2="88.9" y2="160.02" width="0.1524" layer="91"/>
+</segment>
+</net>

Commit message: LED Lib
Parts:
- removed LED1: (no value), led:LED3MM
- added C1: (no value), rcl:C-EUC0805K
- added LED: BLUE, LED-90-Degree:LED-90-DEG
Connections:
- net N$1: now also LED.A; no longer LED1.A
- net N$2: now also LED.C; no longer LED1.C
Changed lines of the file:
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@@
 <part name="ID" library="Right-Angle-Switch" library_urn="urn:adsk.eagle:library:12341455" deviceset="RIGHT-ANGLE-SWITCH" device="" package3d_urn="urn:adsk.eagle:package:12341458/3"/>
 <part name="P5+" library="Female-Header" library_urn="urn:adsk.eagle:library:12344421" deviceset="2PIN-FEMALE-HEADER" device="" package3d_urn="urn:adsk.eagle:package:12344424/3"/>
-<part name="LED1" library="led" library_urn="urn:adsk.eagle:library:259" deviceset="LED" device="3MM" package3d_urn="urn:adsk.eagle:package:15797/1"/>
 <part name="R1" library="rcl" library_urn="urn:adsk.eagle:library:334" deviceset="R-EU_" device="R0805" package3d_urn="urn:adsk.eagle:package:23553/2" value="330R"/>
 <part name="R2" library="rcl" library_urn="urn:adsk.eagle:library:334" deviceset="R-EU_" device="R0805" package3d_urn="urn:adsk.eagle:package:23553/2" value="10K"/>
@@
 <part name="R5" library="rcl" library_urn="urn:adsk.eagle:library:334" deviceset="R-EU_" device="R0805" package3d_urn="urn:adsk.eagle:package:23553/2" value="330R"/>
 <part name="J1" library="con-jack-3D" library_urn="urn:adsk.eagle:library:12345140" deviceset="JACK-PLUG-SLOTTED" device="0" package3d_urn="urn:adsk.eagle:package:12345148/2"/>
+<part name="LED" library="LED-90-Degree" library_urn="urn:adsk.eagle:library:12346089" deviceset="LED-90-DEG" device="" package3d_urn="urn:adsk.eagle:package:12346092/4" value="BLUE"/>
+<part name="C1" library="rcl" library_urn="urn:adsk.eagle:library:334" deviceset="C-EU" device="C0805K" package3d_urn="urn:adsk.eagle:package:23681/2"/>
 </parts>
 <sheets>
@@
 </instance>
 <instance part="P5+" gate="G$1" x="215.9" y="137.16" smashed="yes"/>
-<instance part="LED1" gate="G$1" x="134.62" y="137.16" smashed="yes">
-<attribute name="NAME" x="138.176" y="132.588" size="1.778" layer="95" rot="R90"/>
-<attribute name="VALUE" x="140.335" y="132.588" size="1.778" layer="96" rot="R90"/>
-</instance>
 <instance part="R1" gate="G$1" x="134.62" y="93.98" smashed="yes" rot="R90">
 <attribute name="NAME" x="133.1214" y="90.17" size="1.778" layer="95" rot="R90"/>
@@
 <attribute name="NAME" x="71.12" y="157.48" size="1.778" layer="95"/>
 <attribute name="VALUE" x="71.12" y="147.32" size="1.778" layer="96"/>
+</instance>
+<instance part="LED" gate="G$1" x="134.62" y="134.62" smashed="yes">
+<attribute name="NAME" x="138.176" y="132.588" size="1.778" layer="95" rot="R90"/>
+<attribute name="VALUE" x="140.335" y="132.588" size="1.778" layer="96" rot="R90"/>
+</instance>
+<instance part="C1" gate="G$1" x="116.84" y="149.86" smashed="yes">
+<attribute name="NAME" x="118.364" y="150.241" size="1.778" layer="95"/>
+<attribute name="VALUE" x="118.364" y="145.161" size="1.778" layer="96"/>
 </instance>
 </instances>
@@
 <pinref part="PCB2" gate="G$1" pin="GPIO22"/>
 <wire x1="243.84" y1="152.4" x2="243.84" y2="147.32" width="0.1524" layer="91"/>
-<pinref part="LED1" gate="G$1" pin="A"/>
 <wire x1="243.84" y1="147.32" x2="134.62" y2="147.32" width="0.1524" layer="91"/>
 <wire x1="134.62" y1="147.32" x2="134.62" y2="139.7" width="0.1524" layer="91"/>
+<pinref part="LED" gate="G$1" pin="A"/>
 </segment>
 </net>
 <net name="N$2" class="0">
 <segment>
-<pinref part="LED1" gate="G$1" pin="C"/>
 <pinref part="R1" gate="G$1" pin="2"/>
 <wire x1="134.62" y1="132.08" x2="134.62" y2="99.06" width="0.1524" layer="91"/>
+<pinref part="LED" gate="G$1" pin="C"/>
 </segment>
 </net>
