File: ECAD/KinectIP.sch (EAGLE design)
At the start: 13 parts, among them P5+ 2PIN-FEMALE-HEADER

Commit message: update ECAD
Parts:
- added KINECT_BLACK, KINECT_BROWN, KINECT_GREY, USB3_BLUE, USB3_GND1, USB3_GND2, USB3_ORANGE, USB3_PURPLE, USB3_YELLOW, USB_D+, USB_D-, USB_GND, USB_VCC: (no value), wirepad:SMD2
- added SH1, SH2: GND, wirepad:SMD5
Connections:
- net +12V: now also KINECT_BROWN.P
- net 0V: now also KINECT_BLACK.P, KINECT_GREY.P, SH1.P, SH2.P
Changed lines of the file:
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@@
 </classes>
 <parts>
-<part name="PCB2" library="Rock64" library_urn="urn:adsk.eagle:library:12241252" deviceset="ROCK64" device="ROCK64" package3d_urn="urn:adsk.eagle:package:12239992/2"/>
+<part name="PCB2" library="Rock64" library_urn="urn:adsk.eagle:library:12241252" deviceset="ROCK64" device="ROCK64" package3d_urn="urn:adsk.eagle:package:12239992/3"/>
 <part name="PWR" library="Right-Angle-Switch" library_urn="urn:adsk.eagle:library:12341455" deviceset="RIGHT-ANGLE-SWITCH" device="" package3d_urn="urn:adsk.eagle:package:12341458/3"/>
 <part name="ID" library="Right-Angle-Switch" library_urn="urn:adsk.eagle:library:12341455" deviceset="RIGHT-ANGLE-SWITCH" device="" package3d_urn="urn:adsk.eagle:package:12341458/3"/>
@@
 <part name="C1" library="rcl" library_urn="urn:adsk.eagle:library:334" deviceset="C-EU" device="C0805K" package3d_urn="urn:adsk.eagle:package:23681/2" value="100nF"/>
 <part name="12V-&gt;5V" library="diy-modules" library_urn="urn:adsk.eagle:library:12361804" deviceset="DC-DC-STEP-DOWN-MP1584" device="" package3d_urn="urn:adsk.eagle:package:12362133/2"/>
+<part name="SH1" library="wirepad" library_urn="urn:adsk.eagle:library:412" deviceset="SMD5" device="" package3d_urn="urn:adsk.eagle:package:30841/1" value="GND"/>
+<part name="SH2" library="wirepad" library_urn="urn:adsk.eagle:library:412" deviceset="SMD5" device="" package3d_urn="urn:adsk.eagle:package:30841/1" value="GND"/>
+<part name="USB_VCC" library="wirepad" library_urn="urn:adsk.eagle:library:412" deviceset="SMD2" device="" package3d_urn="urn:adsk.eagle:package:30839/1"/>
+<part name="USB_D-" library="wirepad" library_urn="urn:adsk.eagle:library:412" deviceset="SMD2" device="" package3d_urn="urn:adsk.eagle:package:30839/1"/>
+<part name="USB_D+" library="wirepad" library_urn="urn:adsk.eagle:library:412" deviceset="SMD2" device="" package3d_urn="urn:adsk.eagle:package:30839/1"/>
+<part name="USB_GND" library="wirepad" library_urn="urn:adsk.eagle:library:412" deviceset="SMD2" device="" package3d_urn="urn:adsk.eagle:package:30839/1"/>
+<part name="USB3_ORANGE" library="wirepad" library_urn="urn:adsk.eagle:library:412" deviceset="SMD2" device="" package3d_urn="urn:adsk.eagle:package:30839/1"/>
+<part name="USB3_PURPLE" library="wirepad" library_urn="urn:adsk.eagle:library:412" deviceset="SMD2" device="" package3d_urn="urn:adsk.eagle:package:30839/1"/>
+<part name="USB3_GND1" library="wirepad" library_urn="urn:adsk.eagle:library:412" deviceset="SMD2" device="" package3d_urn="urn:adsk.eagle:package:30839/1"/>
+<part name="USB3_GND2" library="wirepad" library_urn="urn:adsk.eagle:library:412" deviceset="SMD2" device="" package3d_urn="urn:adsk.eagle:package:30839/1"/>
+<part name="USB3_YELLOW" library="wirepad" library_urn="urn:adsk.eagle:library:412" deviceset="SMD2" device="" package3d_urn="urn:adsk.eagle:package:30839/1"/>
+<part name="USB3_BLUE" library="wirepad" library_urn="urn:adsk.eagle:library:412" deviceset="SMD2" device="" package3d_urn="urn:adsk.eagle:package:30839/1"/>
+<part name="KINECT_GREY" library="wirepad" library_urn="urn:adsk.eagle:library:412" deviceset="SMD2" device="" package3d_urn="urn:adsk.eagle:package:30839/1"/>
+<part name="KINECT_BLACK" library="wirepad" library_urn="urn:adsk.eagle:library:412" deviceset="SMD2" device="" package3d_urn="urn:adsk.eagle:package:30839/1"/>
+<part name="KINECT_BROWN" library="wirepad" library_urn="urn:adsk.eagle:library:412" deviceset="SMD2" device="" package3d_urn="urn:adsk.eagle:package:30839/1"/>
+<part name="P+3" library="supply1" library_urn="urn:adsk.eagle:library:371" deviceset="+12V" device=""/>
 </parts>
 <sheets>
@@
 <attribute name="NAME" x="88.9" y="154.94" size="1.778" layer="95"/>
 <attribute name="VALUE" x="88.9" y="152.4" size="1.778" layer="96"/>
+</instance>
+<instance part="SH1" gate="1" x="76.2" y="68.58" smashed="yes" rot="R90">
+<attribute name="NAME" x="74.3458" y="67.437" size="1.778" layer="95" rot="R90"/>
+<attribute name="VALUE" x="79.502" y="67.437" size="1.778" layer="96" rot="R90"/>
+</instance>
+<instance part="SH2" gate="1" x="86.36" y="68.58" smashed="yes" rot="R90">
+<attribute name="NAME" x="84.5058" y="67.437" size="1.778" layer="95" rot="R90"/>
+<attribute name="VALUE" x="89.662" y="67.437" size="1.778" layer="96" rot="R90"/>
+</instance>
+<instance part="USB_VCC" gate="1" x="20.32" y="121.92" smashed="yes">
+<attribute name="NAME" x="19.177" y="123.7742" size="1.778" layer="95"/>
+<attribute name="VALUE" x="19.177" y="118.618" size="1.778" layer="96"/>
+</instance>
+<instance part="USB_D-" gate="1" x="20.32" y="116.84" smashed="yes">
+<attribute name="NAME" x="19.177" y="118.6942" size="1.778" layer="95"/>
+<attribute name="VALUE" x="19.177" y="113.538" size="1.778" layer="96"/>
+</instance>
+<instance part="USB_D+" gate="1" x="20.32" y="111.76" smashed="yes">
+<attribute name="NAME" x="19.177" y="113.6142" size="1.778" layer="95"/>
+<attribute name="VALUE" x="19.177" y="108.458" size="1.778" layer="96"/>
+</instance>
+<instance part="USB_GND" gate="1" x="20.32" y="106.68" smashed="yes">
+<attribute name="NAME" x="19.177" y="108.5342" size="1.778" layer="95"/>
+<attribute name="VALUE" x="19.177" y="103.378" size="1.778" layer="96"/>
+</instance>
+<instance part="USB3_ORANGE" gate="1" x="20.32" y="99.06" smashed="yes">
+<attribute name="NAME" x="19.177" y="100.9142" size="1.778" layer="95"/>
+<attribute name="VALUE" x="19.177" y="95.758" size="1.778" layer="96"/>
+</instance>
+<instance part="USB3_PURPLE" gate="1" x="20.32" y="93.98" smashed="yes">
+<attribute name="NAME" x="19.177" y="95.8342" size="1.778" layer="95"/>
+<attribute name="VALUE" x="19.177" y="90.678" size="1.778" layer="96"/>
+</instance>
+<instance part="USB3_GND1" gate="1" x="20.32" y="88.9" smashed="yes">
+<attribute name="NAME" x="19.177" y="90.7542" size="1.778" layer="95"/>
+<attribute name="VALUE" x="19.177" y="85.598" size="1.778" layer="96"/>
+</instance>
+<instance part="USB3_GND2" gate="1" x="20.32" y="83.82" smashed="yes">
+<attribute name="NAME" x="19.177" y="85.6742" size="1.778" layer="95"/>
+<attribute name="VALUE" x="19.177" y="80.518" size="1.778" layer="96"/>
+</instance>
+<instance part="USB3_YELLOW" gate="1" x="20.32" y="78.74" smashed="yes">
+<attribute name="NAME" x="19.177" y="80.5942" size="1.778" layer="95"/>
+<attribute name="VALUE" x="19.177" y="75.438" size="1.778" layer="96"/>
+</instance>
+<instance part="USB3_BLUE" gate="1" x="20.32" y="73.66" smashed="yes">
+<attribute name="NAME" x="19.177" y="75.5142" size="1.778" layer="95"/>
+<attribute name="VALUE" x="19.177" y="70.358" size="1.778" layer="96"/>
+</instance>
+<instance part="KINECT_GREY" gate="1" x="20.32" y="129.54" smashed="yes">
+<attribute name="NAME" x="19.177" y="131.3942" size="1.778" layer="95"/>
+<attribute name="VALUE" x="19.177" y="126.238" size="1.778" layer="96"/>
+</instance>
+<instance part="KINECT_BLACK" gate="1" x="20.32" y="134.62" smashed="yes">
+<attribute name="NAME" x="19.177" y="136.4742" size="1.778" layer="95"/>
+<attribute name="VALUE" x="19.177" y="131.318" size="1.778" layer="96"/>
+</instance>
+<instance part="KINECT_BROWN" gate="1" x="20.32" y="139.7" smashed="yes">
+<attribute name="NAME" x="19.177" y="141.5542" size="1.778" layer="95"/>
+<attribute name="VALUE" x="19.177" y="136.398" size="1.778" layer="96"/>
+</instance>
+<instance part="P+3" gate="1" x="45.72" y="162.56" smashed="yes">
+<attribute name="VALUE" x="43.18" y="157.48" size="1.778" layer="96" rot="R90"/>
 </instance>
 </instances>
@@
 <wire x1="71.12" y1="149.86" x2="76.2" y2="149.86" width="0.1524" layer="91"/>
 <wire x1="76.2" y1="149.86" x2="76.2" y2="144.78" width="0.1524" layer="91"/>
-<wire x1="76.2" y1="144.78" x2="76.2" y2="71.12" width="0.1524" layer="91"/>
-<wire x1="76.2" y1="71.12" x2="119.38" y2="71.12" width="0.1524" layer="91"/>
+<wire x1="76.2" y1="144.78" x2="76.2" y2="134.62" width="0.1524" layer="91"/>
+<wire x1="76.2" y1="134.62" x2="76.2" y2="129.54" width="0.1524" layer="91"/>
+<wire x1="76.2" y1="129.54" x2="76.2" y2="71.12" width="0.1524" layer="91"/>
+<wire x1="76.2" y1="71.12" x2="86.36" y2="71.12" width="0.1524" layer="91"/>
 <junction x="134.62" y="71.12"/>
 <pinref part="J1" gate="G$1" pin="2"/>
+<wire x1="86.36" y1="71.12" x2="119.38" y2="71.12" width="0.1524" layer="91"/>
 <wire x1="119.38" y1="71.12" x2="127" y2="71.12" width="0.1524" layer="91"/>
 <wire x1="127" y1="71.12" x2="134.62" y2="71.12" width="0.1524" layer="91"/>
@@
 <wire x1="119.38" y1="88.9" x2="119.38" y2="71.12" width="0.1524" layer="91"/>
 <junction x="119.38" y="71.12"/>
+<pinref part="SH1" gate="1" pin="P"/>
+<junction x="76.2" y="71.12"/>
+<pinref part="SH2" gate="1" pin="P"/>
+<junction x="86.36" y="71.12"/>
+<pinref part="KINECT_BLACK" gate="1" pin="P"/>
+<wire x1="22.86" y1="134.62" x2="76.2" y2="134.62" width="0.1524" layer="91"/>
+<junction x="76.2" y="134.62"/>
+<pinref part="KINECT_GREY" gate="1" pin="P"/>
+<wire x1="22.86" y1="129.54" x2="76.2" y2="129.54" width="0.1524" layer="91"/>
+<junction x="76.2" y="129.54"/>
 </segment>
 </net>
@@
 <junction x="83.82" y="137.16"/>
 </segment>
-</net>
+<segment>
+<pinref part="KINECT_BROWN" gate="1" pin="P"/>
+<pinref part="P+3" gate="1" pin="+12V"/>
+<wire x1="22.86" y1="139.7" x2="45.72" y2="139.7" width="0.1524" layer="91"/>
+<wire x1="45.72" y1="139.7" x2="45.72" y2="160.02" width="0.1524" layer="91"/>
+</segment>
+</net>

Commit message: ecad update
Parts:
- added PAD1, PAD2, PAD3, PAD4: (no value), wirepad:1,6/0,8
- added U$1: BOJIT_COPPER, BOJIT Logos:BOJIT_COPPER
- added USB3_BLUE_HOST, USB3_GND1_HOST, USB3_GND2_HOST, USB3_ORANGE_HOST, USB3_PURPLE_HOST, USB3_YELLOW_HOST, USB_D+_HOST, USB_D-_HOST, USB_GND_HOST, USB_VCC_HOST: (no value), wirepad:SMD2
Connections:
- new net N$10: USB_GND.P, USB_GND_HOST.P
- new net N$11: USB3_ORANGE.P, USB3_ORANGE_HOST.P
- new net N$12: USB3_PURPLE.P, USB3_PURPLE_HOST.P
- new net N$13: USB3_GND1.P, USB3_GND1_HOST.P, USB3_GND2.P, USB3_GND2_HOST.P
- new net N$15: USB3_YELLOW.P, USB3_YELLOW_HOST.P
- new net N$16: USB3_BLUE.P, USB3_BLUE_HOST.P
- new net N$7: USB_VCC.P, USB_VCC_HOST.P
- new net N$8: USB_D-.P, USB_D-_HOST.P
- new net N$9: USB_D+.P, USB_D+_HOST.P
Other:
- moved on the sheet: USB3_BLUE, USB3_GND1, USB3_GND2, USB3_ORANGE, USB3_PURPLE, USB3_YELLOW
